File: KOTLETA.brd (EAGLE design)
At the start: 27 x 40.2 mm, 124 parts, among them CON1 CON-6P, CON2 CON-4P-JST_GH-RA, CON3 CON-4P-JST_GH-RA, IC1 STM32F105RCT6, IC2 CAT24C02, IC3 SN65HVD232D, IC4 LMR14010ADDCT, IC5 LM75BD-TSSOP8, IC6 FAN7888, IC7 ZXCT1051, IC8 3.3V, Q1 CSD18510Q5B, Q2 CSD18510Q5B, Q3 CSD18510Q5B, Q4 CSD18510Q5B, Q5 CSD18510Q5B, Q6 CSD18510Q5B, X1 24MHz

Commit message: minor updates
Parts:
- added PAD21, PAD22: PAD-HOLE-0.8, PADS:HOLE_0.8
- moved FD4 18.0 mm to (-2.60, -3.98)
Connections:
- net VDD_9V renamed VDD_10V5
- removed net CAN2_RX: IC1.33
- removed net CAN2_TX: IC1.34
- net GND: now also PAD22.P$1
- net VBAT: now also PAD21.P$1
Changed lines of the file:
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@@
 <drawing>
 <settings>
-<setting alwaysvectorfont="no"/>
+<setting alwaysvectorfont="yes"/>
 <setting keepoldvectorfont="yes"/>
 <setting verticaltext="up"/>
@@
 <grid distance="0.025" unitdist="mm" unit="mm" style="lines" multiple="2" display="yes" altdistance="1" altunitdist="mm" altunit="mm"/>
 <layers>
-<layer number="1" name="Top" color="4" fill="1" visible="yes" active="yes"/>
+<layer number="1" name="Top" color="4" fill="1" visible="no" active="yes"/>
 <layer number="2" name="gnd" color="1" fill="3" visible="no" active="yes"/>
 <layer number="3" name="SUPPLY" color="2" fill="5" visible="no" active="yes"/>
@@
 <layer number="14" name="Horizontal" color="13" fill="1" visible="no" active="no"/>
 <layer number="15" name="+3v3" color="4" fill="6" visible="no" active="no"/>
-<layer number="16" name="Bottom" color="1" fill="1" visible="no" active="yes"/>
+<layer number="16" name="Bottom" color="1" fill="1" visible="yes" active="yes"/>
 <layer number="17" name="Pads" color="2" fill="1" visible="yes" active="yes"/>
 <layer number="18" name="Vias" color="2" fill="1" visible="yes" active="yes"/>
 <layer number="19" name="Unrouted" color="14" fill="1" visible="yes" active="yes"/>
 <layer number="20" name="Dimension" color="15" fill="1" visible="yes" active="yes"/>
-<layer number="21" name="tPlace" color="7" fill="1" visible="yes" active="yes"/>
-<layer number="22" name="bPlace" color="7" fill="1" visible="no" active="yes"/>
-<layer number="23" name="tOrigins" color="15" fill="1" visible="yes" active="yes"/>
-<layer number="24" name="bOrigins" color="15" fill="1" visible="no" active="yes"/>
-<layer number="25" name="tNames" color="7" fill="1" visible="yes" active="yes"/>
-<layer number="26" name="bNames" color="7" fill="1" visible="no" active="yes"/>
+<layer number="21" name="tPlace" color="7" fill="1" visible="no" active="yes"/>
+<layer number="22" name="bPlace" color="7" fill="1" visible="yes" active="yes"/>
+<layer number="23" name="tOrigins" color="15" fill="1" visible="no" active="yes"/>
+<layer number="24" name="bOrigins" color="15" fill="1" visible="yes" active="yes"/>
+<layer number="25" name="tNames" color="7" fill="1" visible="no" active="yes"/>
+<layer number="26" name="bNames" color="7" fill="1" visible="yes" active="yes"/>
 <layer number="27" name="tValues" color="7" fill="1" visible="no" active="yes"/>
 <layer number="28" name="bValues" color="7" fill="1" visible="no" active="yes"/>
@@
 <layer number="49" name="Reference" color="7" fill="1" visible="no" active="yes"/>
 <layer number="50" name="dxf" color="7" fill="1" visible="no" active="no"/>
-<layer number="51" name="tDocu" color="7" fill="1" visible="yes" active="yes"/>
-<layer number="52" name="bDocu" color="7" fill="1" visible="no" active="yes"/>
+<layer number="51" name="tDocu" color="7" fill="1" visible="no" active="yes"/>
+<layer number="52" name="bDocu" color="7" fill="1" visible="yes" active="yes"/>
 <layer number="53" name="tGND_GNDA" color="7" fill="9" visible="no" active="no"/>
 <layer number="54" name="bGND_GNDA" color="1" fill="9" visible="no" active="no"/>
@@
 </layers>
 <board>
-<fusionsync huburn="a.cGVyc29uYWw6dWUyYWE4ZDY4" projecturn="a.cGVyc29uYWw6dWUyYWE4ZDY4IzIwMTkwMjAzMTc0MDAzODgx" f3durn="urn:adsk.wipprod:dm.lineage:CTH-7dBBS_G654204HbCxw" pcbguid="6951ede2-7dc7-4c16-80e3-2d825fdd5a87" lastpulledtime="" lastsyncedchangeguid="3a30d25b-6c2b-df89-f102-d45e4b5ded2e"/>
+<fusionsync huburn="a.cGVyc29uYWw6dWUyYWE4ZDY4" projecturn="a.cGVyc29uYWw6dWUyYWE4ZDY4IzIwMTkwMjAzMTc0MDAzODgx" f3durn="urn:adsk.wipprod:dm.lineage:CTH-7dBBS_G654204HbCxw" pcbguid="6951ede2-7dc7-4c16-80e3-2d825fdd5a87" lastpulledtime="" lastsyncedchangeguid="18577fc7-55b0-ecca-7b5a-7514e5ae479c"/>
 <plain>
 <wire x1="-13.5" y1="18.2" x2="-13.5" y2="19.2" width="0.01" layer="20"/>
@@
 <param name="layerSetup" value="(1+2*3+16)"/>
 <param name="mtCopper" value="0.035mm 0.035mm 0.035mm 0.035mm 0.035mm 0.035mm 0.035mm 0.035mm 0.035mm 0.035mm 0.035mm 0.035mm 0.035mm 0.035mm 0.035mm 0.035mm"/>
-<param name="mtIsolate" value="0.5mm 0.5mm 0.2mm 0.15mm 0.2mm 0.15mm 0.2mm 0.15mm 0.2mm 0.15mm 0.2mm 0.15mm 0.2mm 0.15mm 0.5mm"/>
+<param name="mtIsolate" value="0.012mm 1.5mm 0.012mm 0.15mm 0.2mm 0.15mm 0.2mm 0.15mm 0.2mm 0.15mm 0.2mm 0.15mm 0.2mm 0.15mm 0.5mm"/>
 <param name="mdWireWire" value="0.2mm"/>
 <param name="mdWirePad" value="0.2mm"/>
@@
 </element>
 <element name="FD3" library="sapog_reference_hardware" package="FIDUCIA-MOUNT" value="FIDUCIALMOUNT" x="12.225" y="18" smashed="yes" rot="MR0"/>
-<element name="FD4" library="sapog_reference_hardware" package="FIDUCIA-MOUNT" value="FIDUCIALMOUNT" x="-20.6" y="-3.75" smashed="yes" rot="MR0"/>
+<element name="FD4" library="sapog_reference_hardware" package="FIDUCIA-MOUNT" value="FIDUCIALMOUNT" x="-2.6" y="-3.975" smashed="yes" rot="MR0"/>
 <element name="R26" library="R_digikey" library_urn="urn:adsk.eagle:library:2539499" package="R0402" package3d_urn="urn:adsk.eagle:package:2539512/2" value="200R" x="12.05" y="-3.15" smashed="yes" rot="MR270">
 <attribute name="DIGIKEY#" value="311-200JRCT-ND" x="12.05" y="-3.15" size="1.778" layer="28" rot="MR270" display="off"/>
@@
 <attribute name="VALUE" x="-6.2" y="9.975" size="0.5" layer="28" font="vector" ratio="15" rot="MR270" align="center"/>
 </element>
+<element name="PAD21" library="PADS" library_urn="urn:adsk.eagle:library:3188696" package="HOLE_0.8" value="PAD-HOLE-0.8" x="4.2" y="-5.85" smashed="yes" rot="R90"/>
+<element name="PAD22" library="PADS" library_urn="urn:adsk.eagle:library:3188696" package="HOLE_0.8" value="PAD-HOLE-0.8" x="-4.2" y="-5.85" smashed="yes" rot="R90"/>
 </elements>
 <signals>
@@
 </polygon>
 <wire x1="-13.5" y1="0.425" x2="-13.5" y2="-0.475" width="0.2" layer="1"/>
+<contactref element="PAD21" pad="P$1"/>
 </signal>
 <signal name="FET_A_L">
@@
 <via x="-6.85" y="-1.8" extent="1-16" drill="0.3"/>
 <wire x1="-5.8" y1="-7.6" x2="-6.575" y2="-7.6" width="0.2" layer="16"/>
-<wire x1="-6.575" y1="-7.6" x2="-6.8" y2="-7.375" width="0.2" layer="16"/>
+<wire x1="-6.575" y1="-7.6" x2="-6.85" y2="-7.325" width="0.2" layer="16"/>
 <contactref element="IC4" pad="2"/>
 <contactref element="IC8" pad="1"/>
@@
 <via x="-1.225" y="6.8" extent="1-16" drill="0.3"/>
 <via x="-12.05" y="9.05" extent="1-16" drill="0.3"/>
-<wire x1="-6.8" y1="-7.375" x2="-6.8" y2="-4.2" width="0.2" layer="16"/>
+<wire x1="-6.85" y1="-7.325" x2="-6.85" y2="-4.2" width="0.2" layer="16"/>
 <via x="-1.525" y="-1.05" extent="1-16" drill="0.3"/>
 <via x="-0.85" y="12.6" extent="1-16" drill="0.3"/>
@@
 <via x="-2.775" y="17.7" extent="1-16" drill="0.3" diameter="0.55"/>
 <contactref element="IC1" pad="8"/>
+<contactref element="PAD22" pad="P$1"/>
 </signal>
 <signal name="SENSE_B">
@@
 <signal name="N$43">
 </signal>
-<signal name="CAN2_RX">
-<contactref element="IC1" pad="33"/>
-</signal>
-<signal name="CAN2_TX">
-<contactref element="IC1" pad="34"/>
-</signal>
 <signal name="CAN1_TX">
 <contactref element="IC1" pad="45"/>
@@
 <wire x1="5.75" y1="-1.15" x2="6.825" y2="-1.15" width="0.2" layer="16"/>
 <via x="-5.35" y="-4.775" extent="1-16" drill="0.3"/>
-<wire x1="-5.8" y1="-6.65" x2="-5.35" y2="-6.65" width="0.2" layer="16"/>
-<wire x1="-5.35" y1="-6.65" x2="-5.35" y2="-4.775" width="0.2" layer="16"/>
+<wire x1="-5.8" y1="-6.65" x2="-5.45" y2="-6.65" width="0.2" layer="16"/>
+<wire x1="-5.45" y1="-4.875" x2="-5.35" y2="-4.775" width="0.2" layer="16"/>
+<wire x1="-5.45" y1="-4.875" x2="-5.45" y2="-6.65" width="0.2" layer="16"/>
 <via x="10.5" y="-3.2" extent="1-16" drill="0.3"/>
 <wire x1="10.7" y1="-2.3" x2="11.35" y2="-2.3" width="0.4" layer="16"/>
@@
 <vertex x="-9.575" y="-8.55"/>
 <vertex x="-9.575" y="-12.20720625"/>
-<vertex x="-2.3" y="-12.25"/>
-<vertex x="-2.3" y="-10.1"/>
+<vertex x="-2.15" y="-12.25088125"/>
+<vertex x="-2.15" y="-10.1"/>
 <vertex x="13.45" y="-10.1"/>
 <vertex x="13.45" y="-20.1"/>
@@
 <wire x1="-7.45" y1="7.4" x2="-7.45" y2="7.725" width="0.6" layer="16"/>
 </signal>
-<signal name="VDD_9V">
+<signal name="VDD_10V5">
 <contactref element="L1" pad="P$2"/>
 <contactref element="R27" pad="2"/>
