File: KOTLETA.sch (EAGLE design)
At the start: 126 parts, among them CON1 CON-6P, CON2 CON-4P-JST_GH-RA, CON3 CON-4P-JST_GH-RA, IC1 STM32F105RCT6, IC2 CAT24C02, IC3 SN65HVD232D, IC4 LMR14010ADDCT, IC5 LM75BD-TSSOP8, IC6 FAN7888, IC7 ZXCT1051, IC8 3.3V, Q1 CSD18510Q5B, Q2 CSD18510Q5B, Q3 CSD18510Q5B, Q4 CSD18510Q5B, Q5 CSD18510Q5B, Q6 CSD18510Q5B, X1 24MHz

Commit message: notes
Other:
- note added: "These pads are used to connect BULK CAPACITOR. A good one can be found here https://www.digikey.com/product-detail/en/wurth-electronics-inc/860160574017/732-9555-1-ND/5729493"
- moved on the sheet: PAD21, PAD22
Changed lines of the file:
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@@
 Vout max = 11.06</text>
 <text x="78.74" y="52.07" size="0.635" layer="97">https://docs.google.com/spreadsheets/d/1WwElBVsDBB5yf-5zQ-RQBamWm7rKtQzdxvj4nXSMxlk/edit?usp=sharing</text>
+<text x="139.7" y="30.48" size="1.778" layer="97">These pads are used to connect BULK CAPACITOR.
+A good one can be found here
+https://www.digikey.com/product-detail/en/wurth-electronics-inc/860160574017/732-9555-1-ND/5729493</text>
+<wire x1="124.46" y1="38.1" x2="124.46" y2="7.62" width="0.1524" layer="97" style="shortdash"/>
+<wire x1="124.46" y1="7.62" x2="137.16" y2="7.62" width="0.1524" layer="97" style="shortdash"/>
+<wire x1="137.16" y1="7.62" x2="137.16" y2="38.1" width="0.1524" layer="97" style="shortdash"/>
+<wire x1="137.16" y1="38.1" x2="127" y2="38.1" width="0.1524" layer="97" style="shortdash"/>
+<wire x1="127" y1="38.1" x2="124.46" y2="38.1" width="0.1524" layer="97" style="shortdash"/>
 </plain>
 <instances>
@@
 <attribute name="TOLERANCE" x="141.732" y="63.754" size="0.762" layer="96" rot="R90"/>
 </instance>
-<instance part="PAD21" gate="G$1" x="55.88" y="60.96" smashed="yes" rot="MR0">
-<attribute name="NAME" x="55.88" y="62.23" size="1.27" layer="95" font="vector" ratio="15" rot="MR0" align="center"/>
-</instance>
-<instance part="PAD22" gate="G$1" x="55.88" y="53.34" smashed="yes" rot="MR0">
-<attribute name="NAME" x="55.88" y="54.61" size="1.27" layer="95" font="vector" ratio="15" rot="MR0" align="center"/>
-</instance>
-<instance part="+P13" gate="G$1" x="50.8" y="63.5" smashed="yes">
-<attribute name="VALUE" x="50.8" y="67.056" size="1.27" layer="96" font="vector" ratio="15" align="center"/>
-</instance>
-<instance part="GND46" gate="1" x="50.8" y="48.26" smashed="yes">
-<attribute name="VALUE" x="50.8" y="46.99" size="1.27" layer="96" font="vector" ratio="15" align="center"/>
+<instance part="PAD21" gate="G$1" x="134.62" y="27.94" smashed="yes" rot="MR0">
+<attribute name="NAME" x="134.62" y="29.21" size="1.27" layer="95" font="vector" ratio="15" rot="MR0" align="center"/>
+</instance>
+<instance part="PAD22" gate="G$1" x="134.62" y="20.32" smashed="yes" rot="MR0">
+<attribute name="NAME" x="134.62" y="21.59" size="1.27" layer="95" font="vector" ratio="15" rot="MR0" align="center"/>
+</instance>
+<instance part="+P13" gate="G$1" x="129.54" y="30.48" smashed="yes">
+<attribute name="VALUE" x="129.54" y="34.036" size="1.27" layer="96" font="vector" ratio="15" align="center"/>
+</instance>
+<instance part="GND46" gate="1" x="129.54" y="15.24" smashed="yes">
+<attribute name="VALUE" x="129.54" y="13.97" size="1.27" layer="96" font="vector" ratio="15" align="center"/>
 </instance>
 </instances>
@@
 <segment>
 <pinref part="PAD22" gate="G$1" pin="P$1"/>
-<wire x1="53.34" y1="53.34" x2="50.8" y2="53.34" width="0.1524" layer="91"/>
+<wire x1="132.08" y1="20.32" x2="129.54" y2="20.32" width="0.1524" layer="91"/>
 <pinref part="GND46" gate="1" pin="GND"/>
-<wire x1="50.8" y1="53.34" x2="50.8" y2="50.8" width="0.1524" layer="91"/>
+<wire x1="129.54" y1="20.32" x2="129.54" y2="17.78" width="0.1524" layer="91"/>
 </segment>
 </net>
@@
 <segment>
 <pinref part="PAD21" gate="G$1" pin="P$1"/>
-<wire x1="53.34" y1="60.96" x2="50.8" y2="60.96" width="0.1524" layer="91"/>
+<wire x1="132.08" y1="27.94" x2="129.54" y2="27.94" width="0.1524" layer="91"/>
 <pinref part="+P13" gate="G$1" pin="VBAT"/>
-<wire x1="50.8" y1="60.96" x2="50.8" y2="63.5" width="0.1524" layer="91"/>
-</segment>
-</net>
+<wire x1="129.54" y1="27.94" x2="129.54" y2="30.48" width="0.1524" layer="91"/>
+</segment>
+</net>

Commit message: minor updates
Connections:
- net VDD_9V renamed VDD_10V5
- removed net CAN2_RX: IC1.PB12
- removed net CAN2_TX: IC1.PB13
Other:
- moved on the sheet: PAD21, PAD22
Changed lines of the file:
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@@
-</segment>
-</net>
-<net name="CAN2_RX" class="0">
-<segment>
-<pinref part="IC1" gate="G$1" pin="PB12"/>
-<wire x1="121.92" y1="81.28" x2="124.46" y2="81.28" width="0.1524" layer="91"/>
-<label x="124.46" y="81.28" size="1.27" layer="95" xref="yes"/>
-</segment>
-</net>
-<net name="CAN2_TX" class="0">
-<segment>
-<pinref part="IC1" gate="G$1" pin="PB13"/>
-<wire x1="121.92" y1="83.82" x2="124.46" y2="83.82" width="0.1524" layer="91"/>
-<label x="124.46" y="83.82" size="1.27" layer="95" xref="yes"/>
 </segment>
 </net>
@@
 A good one can be found here
 https://www.digikey.com/product-detail/en/wurth-electronics-inc/860160574017/732-9555-1-ND/5729493</text>
-<wire x1="124.46" y1="38.1" x2="124.46" y2="7.62" width="0.1524" layer="97" style="shortdash"/>
-<wire x1="124.46" y1="7.62" x2="137.16" y2="7.62" width="0.1524" layer="97" style="shortdash"/>
-<wire x1="137.16" y1="7.62" x2="137.16" y2="38.1" width="0.1524" layer="97" style="shortdash"/>
-<wire x1="137.16" y1="38.1" x2="127" y2="38.1" width="0.1524" layer="97" style="shortdash"/>
-<wire x1="127" y1="38.1" x2="124.46" y2="38.1" width="0.1524" layer="97" style="shortdash"/>
+<wire x1="121.92" y1="38.1" x2="121.92" y2="7.62" width="0.1524" layer="97" style="shortdash"/>
+<wire x1="121.92" y1="7.62" x2="134.62" y2="7.62" width="0.1524" layer="97" style="shortdash"/>
+<wire x1="134.62" y1="7.62" x2="134.62" y2="38.1" width="0.1524" layer="97" style="shortdash"/>
+<wire x1="134.62" y1="38.1" x2="124.46" y2="38.1" width="0.1524" layer="97" style="shortdash"/>
+<wire x1="124.46" y1="38.1" x2="121.92" y2="38.1" width="0.1524" layer="97" style="shortdash"/>
 </plain>
 <instances>
@@
 <attribute name="TOLERANCE" x="141.732" y="63.754" size="0.762" layer="96" rot="R90"/>
 </instance>
-<instance part="PAD21" gate="G$1" x="134.62" y="27.94" smashed="yes" rot="MR0">
-<attribute name="NAME" x="134.62" y="29.21" size="1.27" layer="95" font="vector" ratio="15" rot="MR0" align="center"/>
-</instance>
-<instance part="PAD22" gate="G$1" x="134.62" y="20.32" smashed="yes" rot="MR0">
-<attribute name="NAME" x="134.62" y="21.59" size="1.27" layer="95" font="vector" ratio="15" rot="MR0" align="center"/>
-</instance>
-<instance part="+P13" gate="G$1" x="129.54" y="30.48" smashed="yes">
-<attribute name="VALUE" x="129.54" y="34.036" size="1.27" layer="96" font="vector" ratio="15" align="center"/>
-</instance>
-<instance part="GND46" gate="1" x="129.54" y="15.24" smashed="yes">
-<attribute name="VALUE" x="129.54" y="13.97" size="1.27" layer="96" font="vector" ratio="15" align="center"/>
+<instance part="PAD21" gate="G$1" x="132.08" y="27.94" smashed="yes" rot="MR0">
+<attribute name="NAME" x="132.08" y="29.21" size="1.27" layer="95" font="vector" ratio="15" rot="MR0" align="center"/>
+</instance>
+<instance part="PAD22" gate="G$1" x="132.08" y="20.32" smashed="yes" rot="MR0">
+<attribute name="NAME" x="132.08" y="21.59" size="1.27" layer="95" font="vector" ratio="15" rot="MR0" align="center"/>
+</instance>
+<instance part="+P13" gate="G$1" x="127" y="30.48" smashed="yes">
+<attribute name="VALUE" x="127" y="34.036" size="1.27" layer="96" font="vector" ratio="15" align="center"/>
+</instance>
+<instance part="GND46" gate="1" x="127" y="15.24" smashed="yes">
+<attribute name="VALUE" x="127" y="13.97" size="1.27" layer="96" font="vector" ratio="15" align="center"/>
 </instance>
 </instances>
@@
 <segment>
 <pinref part="PAD22" gate="G$1" pin="P$1"/>
-<wire x1="132.08" y1="20.32" x2="129.54" y2="20.32" width="0.1524" layer="91"/>
+<wire x1="129.54" y1="20.32" x2="127" y2="20.32" width="0.1524" layer="91"/>
 <pinref part="GND46" gate="1" pin="GND"/>
-<wire x1="129.54" y1="20.32" x2="129.54" y2="17.78" width="0.1524" layer="91"/>
+<wire x1="127" y1="20.32" x2="127" y2="17.78" width="0.1524" layer="91"/>
 </segment>
 </net>
@@
 <segment>
 <pinref part="PAD21" gate="G$1" pin="P$1"/>
-<wire x1="132.08" y1="27.94" x2="129.54" y2="27.94" width="0.1524" layer="91"/>
+<wire x1="129.54" y1="27.94" x2="127" y2="27.94" width="0.1524" layer="91"/>
 <pinref part="+P13" gate="G$1" pin="VBAT"/>
-<wire x1="129.54" y1="27.94" x2="129.54" y2="30.48" width="0.1524" layer="91"/>
+<wire x1="127" y1="27.94" x2="127" y2="30.48" width="0.1524" layer="91"/>
 </segment>
 </net>
@@
 <segment>
 <pinref part="Q2" gate="G$1" pin="S"/>
-<wire x1="134.62" y1="134.62" x2="134.62" y2="132.08" width="0.1524" layer="91"/>
+<wire x1="134.62" y1="134.62" x2="134.62" y2="109.22" width="0.1524" layer="91"/>
 <pinref part="Q4" gate="G$1" pin="S"/>
 <wire x1="190.5" y1="134.62" x2="190.5" y2="132.08" width="0.1524" layer="91"/>
@@
 <wire x1="190.5" y1="109.22" x2="190.5" y2="96.52" width="0.1524" layer="91"/>
 <junction x="190.5" y="109.22"/>
-<wire x1="134.62" y1="132.08" x2="134.62" y2="109.22" width="0.1524" layer="91"/>
 <wire x1="134.62" y1="109.22" x2="190.5" y2="109.22" width="0.1524" layer="91"/>
 <pinref part="R14" gate="G$1" pin="1"/>
@@
 </segment>
 </net>
-<net name="VDD_9V" class="0">
+<net name="VDD_10V5" class="0">
 <segment>
 <pinref part="L1" gate="G$1" pin="P$2"/>
